File: CANdwich_hub.kicad_sch (KiCad schematic)
At the start: 52 parts, among them J1 USB_C_Receptacle_USB2.0, J2 Conn_01x04_Socket, J3 Conn_01x04_Socket, J4 Conn_01x04_Socket, J5 Conn_01x04_Socket, U1 AP2127K-3.3, U2 USB2514B_Bi, Y1 7U24000E08UCG

Commit message: Footprint placement
Parts:
- removed TP10, TP11, TP4, TP5, TP6, TP7, TP8, TP9: TestPoint, TestPoint:TestPoint_Pad_D1.0mm, symbol Connector:TestPoint
- added H1, H2, H3, H4, H5, H6, H7, H8: MountingHole_Pad, 0_terry:USB_EdgeMount_GND_hub, symbol Mechanical:MountingHole_Pad
- added H10, H11, H12, H9: MountingHole_Pad, 0_terry:USB_EdgeMount_GND_long, symbol Mechanical:MountingHole_Pad
- J2, J3, J4, J5: footprint 0_terry:USB_snowflake -> 0_terry:USB_EdgeMount_Hub
Connections:
- net Earth: now also H1.1, H10.1, H11.1, H12.1, H2.1, H3.1, H4.1, H5.1, H6.1, H7.1, H8.1, H9.1
